Commit message: Payload task

File: payload_code/urdf/hrp4.urdf (robot description, URDF)
Before this commit: robot hrp4, 55 links, 54 joints
Links:
- link L_ELBOW_P_LINK: geometry collision box size=0.1 0.1 0.1; visual mesh filename=../meshes/ELBOW_P.dae
- link L_F23_LINK: geometry collision box size=0.1 0.1 0.1; visual mesh filename=../meshes/F3.dae
- link L_HAND_J0_LINK: geometry collision box size=0.1 0.1 0.1; visual mesh filename=../meshes/L_THUMB.dae
- link L_HAND_J1_LINK: geometry collision box size=0.1 0.1 0.1; visual mesh filename=../meshes/L_F1.dae
- link L_WRIST_P_LINK: geometry collision box size=0.1 0.1 0.1; visual mesh filename=../meshes/WRIST_P.dae
- link R_ELBOW_P_LINK: geometry collision box size=0.1 0.1 0.1; visual mesh filename=../meshes/ELBOW_P.dae
- link R_F23_LINK: geometry collision box size=0.1 0.1 0.1; visual mesh filename=../meshes/F3.dae
- link R_HAND_J0_LINK: geometry collision box size=0.1 0.1 0.1; visual mesh filename=../meshes/R_THUMB.dae
- link R_HAND_J1_LINK: geometry collision box size=0.1 0.1 0.1; visual mesh filename=../meshes/R_F1.dae
- link R_HIP_P_LINK: geometry collision box size=0.1 0.1 0.1; visual mesh filename=../meshes/R_HIP_P.dae
- link R_HIP_R_LINK: geometry collision box size=0.1 0.1 0.1; visual mesh filename=../meshes/CHEST_P.dae
- link R_HIP_Y_LINK: geometry collision box size=0.1 0.1 0.1; visual mesh filename=../meshes/HIP_Y.dae
- link R_WRIST_P_LINK: geometry collision box size=0.1 0.1 0.1; visual mesh filename=../meshes/WRIST_P.dae
- link body: geometry collision box size=0.1 0.1 0.1; visual mesh filename=../meshes/WAIST_LINK.dae
- link torso: geometry collision box size=0.1 0.1 0.1; visual mesh filename=../meshes/CHEST_Y.dae
Joints:
- joint L_ELBOW_P: origin xyz=0 0 -0.283 rpy=0 0 0 -> xyz=0 0 -0.283 rpy=0 -1.7 0; type revolute -> fixed
- joint L_HAND_J1: origin xyz=0 0 -0.111 rpy=0 0 0 -> xyz=0 0 -0.111 rpy=-1.57 0 0
- joint L_SHOULDER_Y: type revolute -> fixed
- joint L_WRIST_Y: origin xyz=0 0 0 rpy=0 0 0 -> xyz=0 0 0 rpy=0 0 1.5
- joint R_ELBOW_P: limit lower=-2.14675494333333 upper=0.0349065844444444 effort=46.99 velocity=2.64940980453 -> lower=-2.14675494333333 upper=0.2 effort=46.99 velocity=2.64940980453; origin xyz=0 0 -0.283 rpy=0 0 0 -> xyz=0 0 -0.283 rpy=0 -1.7 0; type revolute -> fixed
- joint R_HAND_J0: origin xyz=0.03419 0 -0.039 rpy=0 0.4118977034707 0 -> xyz=0.03419 0 -0.039 rpy=1.5707 0.4118977034707 0
- joint R_HAND_J1: origin xyz=0 0 -0.111 rpy=0 0 0 -> xyz=0 0 -0.111 rpy=1.57 0 0
- joint R_WRIST_Y: origin xyz=0 0 0 rpy=0 0 0 -> xyz=0 0 0 rpy=0 0 -1.5
