Commit message: used new mpc for payload

File: payload_code/urdf/box.urdf (robot description, URDF)
Before this commit: robot box, 3 links, 2 joints
Links:
- removed link s_1
- link s_0: mass 0.7 -> 2.25
Joints:
- removed joint joint_s_0_s_1

Commit message: Correct the computation of angular momentum using dartpy API. tuning k1, k2. Max payload achieve is 1.5kg

File: payload_code/urdf/box.urdf (robot description, URDF)
Before this commit: robot box, 2 links, 1 joints
Links:
- link s_0: mass 2.25 -> 1.5

Commit message: minor work

File: payload_code/urdf/box.urdf (robot description, URDF)
Before this commit: robot box, 2 links, 1 joints
Links:
- link s_0: mass 1.5 -> 2.0
